File: ESP32_Cam.kicad_sch (KiCad schematic)
At the start: 1 part, among them U1 ESP32-CAM

Commit message: Newly updated version, should be ready for ordering, ask Colin tomorrow
Parts:
- removed U1: ESP32-CAM, ESP32-CAM:ESP32-CAM, symbol ESP32-CAM:ESP32-CAM
Connections:
- no-connect marks 12 -> 0
