File: _autosave-Main_Drive.kicad_sch (KiCad schematic)
At the start: 43 parts, among them J1 XT30PW-F, J10 Conn_01x02_Pin, J11 USB4120-03-C_REVA, J2 Conn_01x02_Pin, J3 XT30PW-M, J4 XT30PW-F, J5 XT30PW-F, J6 XT30PW-F, J7 Conn_01x02_Pin, J8 Conn_01x02_Pin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

Commit message: Newly updated version, should be ready for ordering, ask Colin tomorrow
Parts:
- removed J11: USB4120-03-C_REVA, USB4120-03-C_REVA:GCT_USB4120-03-C_REVA, symbol USB4120-03-C_REVA:USB4120-03-C_REVA
- added J11: USB4105-GF-A, USB4105-GF-A-Footprint:GCT_USB4105-GF-A, symbol Custom Symbols:USB4105-GF-A
- Accelerometer1: renamed from U3; MANUFACTURER ST Microelectronics -> 511-LSM6DSOXTR
- C1: footprint Capacitor_SMD:C_0402_1005Metric -> Capacitor_SMD:C_0805_2012Metric; MANUFACTURER (none) -> 581-KAF21KR71E225KU
- C11, C14, C3, C4, C5: footprint Capacitor_SMD:C_0402_1005Metric -> Capacitor_SMD:C_0805_2012Metric; MANUFACTURER (none) -> 581-KAM21KR72A104KU
- C12, C2: footprint Capacitor_SMD:C_0402_1005Metric -> Capacitor_SMD:C_0805_2012Metric; MANUFACTURER (none) -> 581-KAF21KR71E105KU
- C13: footprint Capacitor_SMD:C_0402_1005Metric -> Capacitor_SMD:C_0805_2012Metric; MANUFACTURER (none) -> 581-KAF21KR72A104KL
- H1, H2, H3, H4, J10, J2, J7, J8, J9: MANUFACTURER (none) -> -
- J1, J3, J4, J5, J6: MANUFACTURER (none) -> Amass
- R1, R2: footprint Resistor_SMD:R_0402_1005Metric -> Resistor_SMD:R_0805_2012Metric; MANUFACTURER (none) -> ERA-2AED512X
- R10: footprint Resistor_SMD:R_0402_1005Metric -> Resistor_SMD:R_0805_2012Metric; MANUFACTURER (none) -> 652-CR0805FX-5763ELF; Manufacturer (none) -> 652-CR0805FX-5763ELF
- R11: footprint Resistor_SMD:R_0402_1005Metric -> Resistor_SMD:R_0805_2012Metric; MANUFACTURER (none) -> 71-RCS0805470KJNEA
- R12, R13: footprint Resistor_SMD:R_0402_1005Metric -> Resistor_SMD:R_0805_2012Metric; MANUFACTURER (none) -> 667-ERA-6APB103V
- R16: footprint Resistor_SMD:R_0402_1005Metric -> Resistor_SMD:R_0805_2012Metric; MANUFACTURER (none) -> UP6F5110V
- R3: footprint Resistor_SMD:R_0402_1005Metric -> Resistor_SMD:R_0805_2012Metric; MANUFACTURER (none) -> 652-CRT0805AFY-1001E
- R4, R5: footprint Resistor_SMD:R_0402_1005Metric -> Resistor_SMD:R_0805_2012Metric; MANUFACTURER (none) -> 667-ERA-6APB103V; Manufacturer (none) -> 667-ERA-6APB103V
- renumbered U2 to LDO1, U4 to MCU1
Connections:
- net +V_USB: now also J11.A4_B9 (VBUS), J11.B4_A9 (VBUS)
- net DN: now also J11.A7 (DN1), J11.B7 (DN2)
- net DP: now also J11.A6 (DP1), J11.B6 (DP2)
- net GND: now also J11.A1_B12 (GND), J11.B1_A12 (GND), J11.S1 (SHELL_GND), J11.S2 (SHELL_GND), J11.S3 (SHELL_GND), J11.S4 (SHELL_GND)
- net INT1: now also MCU1.34 (IO38); no longer MCU1.12 (IO8)
- net INT2: now also MCU1.33 (IO37); no longer MCU1.15 (IO11)
- net SCL: now also MCU1.32 (IO36); no longer MCU1.14 (IO10)
- net SDA: now also MCU1.31 (IO35); no longer MCU1.13 (IO9)
- net at C5.1, R10.2, R11.1: now also MCU1.11 (IO7); no longer MCU1.8 (IO4)
- net at R1.1: now also J11.B5 (CC2)
- net at R2.1: now also J11.A5 (CC1)
- net 3_mot: now reaches MCU1.35 (IO39)
- net 3_mot: now also J7.1 (Pin_1)
- net 4_mot: now reaches MCU1.36 (IO40)
- net 4_mot: now also J2.1 (Pin_1)
- net d_motor: no longer names the net of MCU1.22 (IO18)
- net d_motor: no longer J9.1 (Pin_1)
- net d_motor_2: no longer names the net of MCU1.21 (IO17)
- net d_motor_2: no longer J8.1 (Pin_1)
- net l_motor: no longer names the net of MCU1.28 (IO33)
- net l_motor: no longer J7.1 (Pin_1)
- net r_motor: no longer names the net of MCU1.29 (IO34)
- net r_motor: no longer J2.1 (Pin_1)
- new net 1_mot: J8.1 (Pin_1), MCU1.14 (IO10)
- new net 2_mot: J9.1 (Pin_1), MCU1.15 (IO11)
Other:
- note added: "USB C"
- moved on the sheet: C5, R10, R11
