File: BattleBot.kicad_pcb (KiCad board)
At the start: 2 copper layers, 60 x 60.8 mm, 44 parts, among them J1 XT30PW-F, J10 Conn_01x02_Pin, J11 USB4120-03-C_REVA, J2 Conn_01x02_Pin, J3 XT30PW-M, J4 XT30PW-F, J5 XT30PW-F, J6 XT30PW-F, J7 Conn_01x02_Pin, J8 Conn_01x02_Pin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

Commit message: Newly updated version, should be ready for ordering, ask Colin tomorrow
Parts:
- removed G***: LOGO, bitmaps:knife_win_10x13
- removed U2: TLV76601QWDRBRQ1, TLV76601:DRB0008J-IPC_A
- removed U3: LSM6DSOXTR, LSM6DSOXTR:PQFN50P250X300X86-14N
- removed U4: ESP32-S3-MINI-1-N8, esp32s3mini:XCVR_ESP32-S3-MINI-1-N8
- added Accelerometer1: LSM6DSOXTR, LSM6DSOXTR:PQFN50P250X300X86-14N, F.Cu at (227.2, 105.5)
- added LDO1: TLV76601QWDRBRQ1, TLV76601:DRB0008J-IPC_A, F.Cu at (213.5, 100.6)
- added MCU1: ESP32-S3-MINI-1-N8, esp32s3mini:XCVR_ESP32-S3-MINI-1-N8, F.Cu at (218.8, 73.0)
- C1, C11, C12, C13, C14, C2, C3, C4, C5: footprint Capacitor_SMD:C_0402_1005Metric -> Capacitor_SMD:C_0805_2012Metric
- J11: value USB4120-03-C_REVA -> USB4105-GF-A; footprint USB4120-03-C_REVA:GCT_USB4120-03-C_REVA -> USB4105-GF-A-Footprint:GCT_USB4105-GF-A
- R1, R10, R11, R12, R13, R16, R2, R3, R4, R5: footprint Resistor_SMD:R_0402_1005Metric -> Resistor_SMD:R_0805_2012Metric
- moved J5 93.8 mm to (245.0, 82.0), turned to -90 degrees
- moved J6 91.9 mm to (245.0, 96.5), turned to -90 degrees
- moved H1 89.2 mm to (243.0, 115.0)
- moved R16 69.8 mm to (231.3, 113.0), turned to 0 degrees
- moved D2 68.3 mm to (231.3, 116.0), turned to 0 degrees
- moved C3 68.1 mm to (231.2, 108.0), turned to 0 degrees
- moved SW1 66.5 mm to (233.0, 63.2)
- moved C4 65.5 mm to (227.2, 109.5), turned to 180 degrees
- moved R3 63.0 mm to (231.2, 105.0), turned to 0 degrees
- moved R4 61.2 mm to (231.2, 102.5), turned to 0 degrees
- moved R5 55.0 mm to (223.2, 102.5), turned to 180 degrees
- moved C5 47.9 mm to (211.5, 90.0)
- moved C14 46.1 mm to (215.6, 90.0)
- moved SW4 45.9 mm to (213.5, 86.0)
- moved C13 45.6 mm to (215.6, 94.0)
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Connections:
- J1 pad S1: (no net) -> unconnected-(J1-PadS1)
- J1 pad S2: (no net) -> unconnected-(J1-PadS2)
- J2 pad 1: /Main Drive /r_motor -> /Main Drive /4_mot
- J3 pad S1: (no net) -> unconnected-(J3-PadS1)
- J3 pad S2: (no net) -> unconnected-(J3-PadS2)
- J4 pad S1: (no net) -> unconnected-(J4-PadS1)
- J4 pad S2: (no net) -> unconnected-(J4-PadS2)
- J5 pad S1: (no net) -> unconnected-(J5-PadS1)
- J5 pad S2: (no net) -> unconnected-(J5-PadS2)
- J6 pad S1: (no net) -> unconnected-(J6-PadS1)
- J6 pad S2: (no net) -> unconnected-(J6-PadS2)
- J7 pad 1: /Main Drive /l_motor -> /Main Drive /3_mot
- J8 pad 1: /Main Drive /d_motor_2 -> /Main Drive /1_mot
- J9 pad 1: /Main Drive /d_motor -> /Main Drive /2_mot
Routing:
- net /Main Drive /d_motor_2: track 66.0 -> 0.00 mm
- net /Main Drive /r_motor: track 64.2 -> 0.00 mm
- net +BATT: track 76.4 -> 127.7 mm, vias 0 -> 4
- net /Main Drive /2_mot: track 0.00 -> 48.5 mm
- net /Main Drive /3_mot: track 0.00 -> 47.6 mm
- net Net-(SW1-B): track 15.3 -> 60.0 mm, vias 1 -> 4
- net /Main Drive /INT1: track 10.5 -> 50.6 mm, vias 0 -> 2
- net +3V3: track 95.8 -> 131.1 mm, vias 6 -> 3
- net /Main Drive /SDA: track 6.63 -> 38.9 mm
- net /Main Drive /INT2: track 10.2 -> 42.5 mm
- net /Main Drive /SCL: track 7.31 -> 38.9 mm
- net /Main Drive /EN: track 5.15 -> 36.2 mm, vias 0 -> 2
- net /Main Drive /Boot: track 5.21 -> 31.1 mm
- net /Main Drive /d_motor: track 25.0 -> 0.00 mm
- net /Main Drive /1_mot: track 0.00 -> 25.0 mm
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- added copper zone on F.Cu, net Net-(D1-K)
- removed copper zone on F.Cu, net +BATT
Other:
- board size 60 x 60.8 mm -> 60 x 60 mm
- board text added: "JLCJLCJLCJLC"
- board text removed: "REDO PIN LOCATION - BLOCKED BY DRUM MOTOR"
- board text removed: "USE VERTICAL USB-C/SWITCH"

Commit message: 9/29 Ordered PCB
Parts:
- removed SW1: SW_SPDT, JS102011JAQN:SW_JS102011JAQN
- added Q1: PMOS, Package_SO:PowerPAK_SO-8_Single, F.Cu at (233.0, 70.8)
- added R6: 500k, Resistor_SMD:R_0402_1005Metric, F.Cu at (237.5, 68.1)
- added SW2: SW_Nidec_CAS-120A1, Button_Switch_SMD:SW_DPDT_CK_JS202011JCQN, F.Cu at (233.0, 63.0)
Routing:
- net Net-(Q1-G): track 0.00 -> 12.9 mm
- net +BATT: track 127.7 -> 120.6 mm, vias 4 -> 12
- net Net-(SW2A-A): track 60.0 -> 65.6 mm
- net GND: vias 106 -> 96
- added copper zone on F.Cu, net Net-(SW2A-A)

Commit message: OKAY THIS ONE IS THE ORDERED ONE
Connections:
- MCU1 pad 33: /Main Drive /INT2 -> /Main Drive /3_mot
- MCU1 pad 34: /Main Drive /INT1 -> /Main Drive /4_mot
- MCU1 pad 35: /Main Drive /3_mot -> /Main Drive /INT2
- MCU1 pad 36: /Main Drive /4_mot -> /Main Drive /INT1
Routing:
- net +BATT: track 120.6 -> 126.4 mm, vias 12 -> 14
- net /Main Drive /3_mot: track 47.6 -> 48.4 mm, vias 0 -> 2
- net /Main Drive /4_mot: track 22.2 -> 23.0 mm
- net /Main Drive /INT2: track 42.5 -> 43.2 mm
- net /Main Drive /INT1: track 50.6 -> 51.2 mm
